File: pcb/Tx_mother_board/Tx_mother_board/Tx_mother_board.sch (KiCad schematic (older format))
At the start: 17 parts

Commit message: Started aading components schematics to PumaTX KiCAD's library
Parts:
- added P?: ufl, symbol PumaTx:ufl
Changed lines of the file:
@@
 encoding utf-8
 Sheet 1 1
-Title ""
-Date ""
-Rev ""
+Title "PumaTX_MB_HW00"
+Date "2021-05-10"
+Rev "HW00"
 Comp ""
 Comment1 ""
 Comment2 ""
 Comment3 ""
-Comment4 ""
+Comment4 "Author: Nicolas de Grave"
 $EndDescr
 $Comp
@@
 	1    0    0    -1
 $EndComp
+$Comp
+L PumaTx:ufl P?
+U 1 1 609A5838
+P 1750 1950
+F 0 "P?" H 1816 1659 50  0000 R CNN
+F 1 "ufl" H 1816 1750 50  0000 R CNN
+F 2 "" H 2050 2200 50  0001 C CNN
+F 3 "" H 2050 2200 50  0001 C CNN
+	1    1750 1950
+	-1   0    0    1
+$EndComp
+$Comp
+L power:GND #PWR?
+U 1 1 609A684E
+P 1400 1950
+F 0 "#PWR?" H 1400 1700 50  0001 C CNN
+F 1 "GND" V 1405 1822 50  0000 R CNN
+F 2 "" H 1400 1950 50  0001 C CNN
+F 3 "" H 1400 1950 50  0001 C CNN
+	1    1400 1950
+	0    1    1    0
+$EndComp
 $EndSCHEMATC
