File: Hardware/PumaTX_MB_HW00/_autosave-PumaTX_MB_HW00.kicad_sch (KiCad schematic)
At the start: 107 parts, among them J100 FH12A-26S-0.5SH_55_, J101 FH12-12S-0.5SH_55_, J102 500334-0160, J103 500334-0160, J104 692122030100, J105 53398-0667, J300 U.FL-R-SMT-1_40_, J410 U.FL-R-SMT-1_40_, M130 Motor_DC, M140 Fan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

Commit message: Continued routing
Connections:
- net SYS is gone; now on net VSYS: R506.1, R507.1
Changed lines of the file:
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@@
     (effects (font (size 1.27 1.27)) (justify right bottom))
   )
-  (label "SYS" (at 449.58 269.24 0)
+  (label "VSYS" (at 449.58 269.24 0)
     (effects (font (size 1.27 1.27)) (justify left bottom))
   )
